Commit message: First successful implementation. MC without exploring starts Complete

File: bot/.ipynb_checkpoints/robot-checkpoint.urdf (robot description, URDF)
Before this commit: robot onshape, 5 links, 4 joints
Joints:
- joint gripper_2: limit lower=-0.52359877559829881566 upper=0.26179938779914940783 effort=1 velocity=20 -> lower=-0.52359877559829881566 upper=0.36179938779914940783 effort=1 velocity=20
- joint gripper_front: limit lower=-0.52359877559829881566 upper=0.26179938779914940783 effort=1 velocity=20 -> lower=-0.52359877559829881566 upper=0.36179938779914940783 effort=1 velocity=20
- joint slider: limit lower=-0.20999999999999999223 upper=0.23000000000000000999 effort=1 velocity=20 -> lower=-0.210000000000000000 upper=0.21000000000000000999 effort=1 velocity=20

File: bot/robot.urdf (robot description, URDF)
Before this commit: robot onshape, 5 links, 4 joints
Joints:
- joint gripper_2: limit lower=-0.52359877559829881566 upper=0.26179938779914940783 effort=1 velocity=20 -> lower=-0.52359877559829881566 upper=0.36179938779914940783 effort=1 velocity=20
- joint gripper_front: limit lower=-0.52359877559829881566 upper=0.26179938779914940783 effort=1 velocity=20 -> lower=-0.52359877559829881566 upper=0.36179938779914940783 effort=1 velocity=20
- joint slider: limit lower=-0.20999999999999999223 upper=0.23000000000000000999 effort=1 velocity=20 -> lower=-0.210000000000000000 upper=0.21000000000000000999 effort=1 velocity=20
